File: docs/assets/designs/hexapod_circuit/01_battery_protection.kicad_sch (KiCad schematic)
At the start: 3 parts, among them J1 XT90S to battery, SW1 SW_SPST

Commit message: Add files via upload
Changed lines of the file:
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@@
-		)
-	)
-	(label "GND_PWR"
-		(at 38.1 19.05 0)
-		(effects
-			(font
-				(size 1.27 1.27)
-			)
-			(justify left bottom)
 		)
 	)
@@
 		)
 	)
-	(label "V_BAT_SW"
+	(global_label "V_BAT_SW"
+		(shape input)
 		(at 76.2 16.51 0)
+		(fields_autoplaced yes)
 		(effects
 			(font
 				(size 1.27 1.27)
 			)
-			(justify left bottom)
+			(justify left)
+		)
+		(property "Intersheetrefs" "${INTERSHEET_REFS}"
+			(at 88.1961 16.51 0)
+			(effects
+				(font
+					(size 1.27 1.27)
+				)
+				(justify left)
+				(hide yes)
+			)
 		)
 	)
+	(global_label "GND_PWR"
+		(shape input)
+		(at 38.1 19.05 0)
+		(fields_autoplaced yes)
+		(effects
+			(font
+				(size 1.27 1.27)
+			)
+			(justify left)
+		)
+		(property "Intersheetrefs" "${INTERSHEET_REFS}"
+			(at 49.9147 19.05 0)
+			(effects
+				(font
+					(size 1.27 1.27)
+				)
+				(justify left)
+				(hide yes)
+			)
+		)
+	)

Commit message: upload latest schematic version
Parts:
- F1: value 80A ANL -> 120a ANL
- J1: value XT90S to battery -> SB120 to battery
Changed lines of the file:
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@@
 	(generator_version "9.0")
 	(paper "A4")
+	(text_box "X12-320 Has max cont. current of 18.75 A per unit\n\nJetson Nano and connected D415 max of 4 A\n\nESP32 max 500 mA\n\nFSR circuit max 500 uA assuming contact force on FSR does not exceed resistance of 1 kiloohm\n\nThis is about 42 A, assuming a power spike from motor factor of 3, such is a current of 117A\n\nThus we select a 120A ANL fuse as it is the closest to such a value. \n\nThis pairs well with a SB120 connector with max current of 120A"
+		(exclude_from_sim no)
+		(at 12.7 25.4 0)
+		(size 99.06 27.94)
+		(margins 0.9525 0.9525 0.9525 0.9525)
+		(stroke
+			(width 0)
+			(type solid)
+		)
+		(fill
+			(type none)
+		)
+		(effects
+			(font
+				(size 1.27 1.27)
+			)
+			(justify left top)
+		)
+	)
 	(wire
 		(pts
@@
 			)
 		)
-		(property "Value" "80A ANL"
+		(property "Value" "120a ANL"
 			(at 54.356 18.796 90)
 			(effects
@@
 			)
 		)
-		(property "Value" "XT90S to battery"
+		(property "Value" "SB120 to battery"
 			(at 29.21 19.0499 0)
 			(effects
