File: docs/assets/designs/hexapod_circuit/03_DCDC_5V_3.3V.kicad_sch (KiCad schematic)
At the start: 7 parts, among them U1 TRI20-2411, U2 TPS7A0518PDBZ

Commit message: Add files via upload
Other:
- moved on the sheet: C3, C4, U2
Changed lines of the file:
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@@
 	(paper "A4")
 	(junction
-		(at 40.64 36.83)
+		(at 43.18 39.37)
 		(diameter 0)
 		(color 0 0 0 0)
 	)
 	(junction
-		(at 25.4 29.21)
+		(at 27.94 31.75)
 		(diameter 0)
 		(color 0 0 0 0)
@@
 	)
 	(junction
-		(at 25.4 36.83)
+		(at 27.94 39.37)
 		(diameter 0)
 		(color 0 0 0 0)
@@
 	)
 	(junction
-		(at 49.53 29.21)
+		(at 52.07 31.75)
 		(diameter 0)
 		(color 0 0 0 0)
@@
 	(wire
 		(pts
-			(xy 48.26 29.21) (xy 49.53 29.21)
-		)
-		(stroke
-			(width 0)
-			(type default)
-		)
-	)
-	(wire
-		(pts
-			(xy 49.53 29.21) (xy 50.8 29.21)
-		)
-		(stroke
-			(width 0)
-			(type default)
-		)
-	)
-	(wire
-		(pts
-			(xy 25.4 29.21) (xy 33.02 29.21)
+			(xy 50.8 31.75) (xy 52.07 31.75)
+		)
+		(stroke
+			(width 0)
+			(type default)
+		)
+	)
+	(wire
+		(pts
+			(xy 52.07 31.75) (xy 53.34 31.75)
+		)
+		(stroke
+			(width 0)
+			(type default)
+		)
+	)
+	(wire
+		(pts
+			(xy 27.94 31.75) (xy 35.56 31.75)
 		)
 		(stroke
@@
 	(wire
 		(pts
-			(xy 25.4 36.83) (xy 40.64 36.83)
+			(xy 27.94 39.37) (xy 43.18 39.37)
 		)
 		(stroke
@@
 	(wire
 		(pts
-			(xy 24.13 36.83) (xy 25.4 36.83)
+			(xy 26.67 39.37) (xy 27.94 39.37)
 		)
 		(stroke
@@
 	(wire
 		(pts
-			(xy 24.13 29.21) (xy 25.4 29.21)
-		)
-		(stroke
-			(width 0)
-			(type default)
-		)
-	)
-	(wire
-		(pts
-			(xy 40.64 36.83) (xy 49.53 36.83)
+			(xy 26.67 31.75) (xy 27.94 31.75)
+		)
+		(stroke
+			(width 0)
+			(type default)
+		)
+	)
+	(wire
+		(pts
+			(xy 43.18 39.37) (xy 52.07 39.37)
 		)
 		(stroke
@@
 			(width 0)
 			(type default)
-		)
-	)
-	(label "+5V_MAIN"
-		(at 24.13 29.21 180)
-		(effects
-			(font
-				(size 1.27 1.27)
-			)
-			(justify right bottom)
 		)
 	)
@@
 		)
 	)
-	(label "+5V_MAIN"
-		(at 95.25 17.78 0)
-		(effects
-			(font
-				(size 1.27 1.27)
-			)
-			(justify left bottom)
-		)
-	)
-	(label "+3V3_A"
-		(at 50.8 29.21 0)
-		(effects
-			(font
-				(size 1.27 1.27)
-			)
-			(justify left bottom)
-		)
-	)
 	(label "GND_PWR"
 		(at 45.72 22.86 180)
@@
 		)
 	)
-	(label "GND_ELEC"
-		(at 24.13 36.83 180)
+	(global_label "+5V_MAIN"
+		(shape input)
+		(at 95.25 17.78 0)
+		(fields_autoplaced yes)
 		(effects
 			(font
 				(size 1.27 1.27)
 			)
-			(justify right bottom)
-		)
-	)
-	(label "GND_ELEC"
-		(at 95.25 25.4 0)
+			(justify left)
+		)
+		(property "Intersheetrefs" "${INTERSHEET_REFS}"
+			(at 107.5486 17.78 0)
+			(effects
+				(font
+					(size 1.27 1.27)
+				)
+				(justify left)
+				(hide yes)
+			)
+		)
+	)
+	(global_label "GND_ELEC"
+		(shape input)
+		(at 26.67 39.37 180)
+		(fields_autoplaced yes)
 		(effects
 			(font
 				(size 1.27 1.27)
 			)
-			(justify left bottom)
-		)
-	)
-	(label "V_BAT_SW"
+			(justify right)
+		)
+		(property "Intersheetrefs" "${INTERSHEET_REFS}"
+			(at 14.2506 39.37 0)
+			(effects
+				(font
+					(size 1.27 1.27)
+				)
+				(justify right)
+				(hide yes)
+			)
+		)
+	)
+	(global_label "V_BAT_SW"
+		(shape input)
 		(at 24.13 17.78 180)
+		(fields_autoplaced yes)
 		(effects
 			(font
 				(size 1.27 1.27)
 			)
-			(justify right bottom)
+			(justify right)
+		)
+		(property "Intersheetrefs" "${INTERSHEET_REFS}"
+			(at 12.1339 17.78 0)
+			(effects
+				(font
+					(size 1.27 1.27)
+				)
+				(justify right)
+				(hide yes)
+			)
+		)
+	)
+	(global_label "+5V_MAIN"
+		(shape input)
+		(at 26.67 31.75 180)
+		(fields_autoplaced yes)
+		(effects
+			(font
+				(size 1.27 1.27)
+			)
+			(justify right)
+		)
+		(property "Intersheetrefs" "${INTERSHEET_REFS}"
+			(at 14.3714 31.75 0)
+			(effects
+				(font
+					(size 1.27 1.27)
+				)
+				(justify right)
+				(hide yes)
+			)
+		)
+	)
+	(global_label "GND_ELEC"
+		(shape input)
+		(at 95.25 25.4 0)
+		(fields_autoplaced yes)
+		(effects
+			(font
+				(size 1.27 1.27)
+			)
+			(justify left)
+		)
+		(property "Intersheetrefs" "${INTERSHEET_REFS}"
+			(at 107.6694 25.4 0)
+			(effects
+				(font
+					(size 1.27 1.27)
+				)
+				(justify left)
+				(hide yes)
+			)
+		)
+	)
+	(global_label "+3V3_A"
+		(shape input)
+		(at 53.34 31.75 0)
+		(fields_autoplaced yes)
+		(effects
+			(font
+				(size 1.27 1.27)
+			)
+			(justify left)
+		)
+		(property "Intersheetrefs" "${INTERSHEET_REFS}"
+			(at 63.4614 31.75 0)
+			(effects
+				(font
+					(size 1.27 1.27)
+				)
+				(justify left)
+				(hide yes)
+			)
 		)
 	)
@@
 	(symbol
 		(lib_id "Device:C")
-		(at 25.4 33.02 0)
+		(at 27.94 35.56 0)
 		(unit 1)
 		(exclude_from_sim no)
@@
 		(fields_autoplaced yes)
 		(property "Reference" "C3"
-			(at 29.21 31.7499 0)
+			(at 31.75 34.2899 0)
 			(effects
 				(font
@@
 		)
 		(property "Value" "10 µF"
-			(at 29.21 34.2899 0)
+			(at 31.75 36.8299 0)
 			(effects
 				(font
@@
 		)
 		(property "Footprint" ""
-			(at 26.3652 36.83 0)
+			(at 28.9052 39.37 0)
 			(effects
 				(font
@@
 		)
 		(property "Datasheet" "~"
-			(at 25.4 33.02 0)
+			(at 27.94 35.56 0)
 			(effects
 				(font
@@
 		)
 		(property "Description" "Unpolarized capacitor"
-			(at 25.4 33.02 0)
+			(at 27.94 35.56 0)
 			(effects
 				(font
@@
 	(symbol
 		(lib_id "Regulator_Linear:TPS7A0518PDBZ")
-		(at 40.64 29.21 0)
+		(at 43.18 31.75 0)
 		(unit 1)
 		(exclude_from_sim no)
@@
 		(dnp no)
 		(property "Reference" "U2"
-			(at 40.894 25.654 0)
+			(at 43.434 28.194 0)
 			(effects
 				(font
@@
 		)
 		(property "Value" "TPS7A0518PDBZ"
-			(at 40.64 25.4 0)
+			(at 43.18 27.94 0)
 			(effects
 				(font
@@
 		)
 		(property "Footprint" "Package_TO_SOT_SMD:SOT-23"
-			(at 40.64 24.13 0)
+			(at 43.18 26.67 0)
 			(effects
 				(font
@@
 		)
 		(property "Datasheet" "https://www.ti.com/lit/ds/symlink/tps7a05.pdf"
-			(at 40.64 30.48 0)
+			(at 43.18 33.02 0)
 			(effects
 				(font
@@
 		)
 		(property "Description" "200-mA Ultra-Low-Iq LDO, 1.8V, SOT-23-3"
-			(at 40.64 29.21 0)
+			(at 43.18 31.75 0)
 			(effects
 				(font
@@
 	(symbol
 		(lib_id "Device:C")
-		(at 49.53 33.02 0)
+		(at 52.07 35.56 0)
 		(unit 1)
 		(exclude_from_sim no)
@@
 		(fields_autoplaced yes)
 		(property "Reference" "C4"
-			(at 53.34 31.7499 0)
+			(at 55.88 34.2899 0)
 			(effects
 				(font
@@
 		)
 		(property "Value" "10 µF"
-			(at 53.34 34.2899 0)
+			(at 55.88 36.8299 0)
 			(effects
 				(font
@@
 		)
 		(property "Footprint" ""
-			(at 50.4952 36.83 0)
+			(at 53.0352 39.37 0)
 			(effects
 				(font
@@
 		)
 		(property "Datasheet" "~"
-			(at 49.53 33.02 0)
+			(at 52.07 35.56 0)
 			(effects
 				(font
@@
 		)
 		(property "Description" "Unpolarized capacitor"
-			(at 49.53 33.02 0)
-			(effects
-				(font
+			(at 52.07 35.56 0)
+			(effects
+				(font

Commit message: upload latest schematic version
Parts:
- C1: value 1000 µF -> 1 mF
Changed lines of the file:
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@@
 			)
 		)
-		(property "Value" "1000 µF"
+		(property "Value" "1 mF"
 			(at 74.93 23.1139 0)
 			(effects
