File: docs/assets/designs/hexapod_circuit/04_compute_usb.kicad_sch (KiCad schematic)
At the start: 1 part, among them J4 Barrel_Jack_to_Jetson

Commit message: Add files via upload
Other:
- moved on the sheet: J4
Changed lines of the file:
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@@
 	(wire
 		(pts
-			(xy 22.86 21.59) (xy 24.13 21.59)
+			(xy 26.67 21.59) (xy 27.94 21.59)
 		)
 		(stroke
@@
 	(wire
 		(pts
-			(xy 22.86 16.51) (xy 24.13 16.51)
+			(xy 26.67 16.51) (xy 27.94 16.51)
 		)
 		(stroke
@@
 		)
 	)
-	(label "GND_ELEC"
-		(at 22.86 16.51 180)
+	(global_label "GND_ELEC"
+		(shape input)
+		(at 26.67 16.51 180)
+		(fields_autoplaced yes)
 		(effects
 			(font
 				(size 1.27 1.27)
 			)
-			(justify right bottom)
+			(justify right)
+		)
+		(property "Intersheetrefs" "${INTERSHEET_REFS}"
+			(at 14.2506 16.51 0)
+			(effects
+				(font
+					(size 1.27 1.27)
+				)
+				(justify right)
+				(hide yes)
+			)
 		)
 	)
-	(label "+5V_MAIN"
-		(at 22.86 21.59 180)
+	(global_label "+5V_MAIN"
+		(shape input)
+		(at 26.67 21.59 180)
+		(fields_autoplaced yes)
 		(effects
 			(font
 				(size 1.27 1.27)
 			)
-			(justify right bottom)
+			(justify right)
+		)
+		(property "Intersheetrefs" "${INTERSHEET_REFS}"
+			(at 14.3714 21.59 0)
+			(effects
+				(font
+					(size 1.27 1.27)
+				)
+				(justify right)
+				(hide yes)
+			)
 		)
 	)
 	(symbol
 		(lib_id "Connector:Barrel_Jack")
-		(at 31.75 19.05 180)
+		(at 35.56 19.05 180)
 		(unit 1)
 		(exclude_from_sim no)
@@
 		(fields_autoplaced yes)
 		(property "Reference" "J4"
-			(at 38.1 17.7799 0)
+			(at 41.91 17.7799 0)
 			(effects
 				(font
@@
 		)
 		(property "Value" "Barrel_Jack_to_Jetson"
-			(at 38.1 20.3199 0)
+			(at 41.91 20.3199 0)
 			(effects
 				(font
@@
 		)
 		(property "Footprint" ""
-			(at 30.48 18.034 0)
+			(at 34.29 18.034 0)
 			(effects
 				(font
@@
 		)
 		(property "Datasheet" "~"
-			(at 30.48 18.034 0)
+			(at 34.29 18.034 0)
 			(effects
 				(font
@@
 		)
 		(property "Description" "DC Barrel Jack"
-			(at 31.75 19.05 0)
+			(at 35.56 19.05 0)
 			(effects
 				(font

Commit message: upload latest schematic version
Parts:
- added J5: Jetson Nano J41 GPIO, symbol Connector_Generic:Conn_02x20_Top_Bottom
- added J6: LCD1602, symbol Connector_Generic:Conn_01x16
Connections:
- net +5V_MAIN: now also J6.15 (Pin_15)
- net GND_ELEC: now also J6.1 (Pin_1), J6.16 (Pin_16)
- new net +3V3_A: J6.2 (Pin_2)
- new net D0: J6.10 (Pin_10)
- new net D1: J6.9 (Pin_9)
- new net D2: J6.8 (Pin_8)
- new net D3: J6.7 (Pin_7)
- new net D4: J6.6 (Pin_6)
- new net D5: J6.5 (Pin_5)
- new net D6: J6.4 (Pin_4)
- new net D7: J6.3 (Pin_3)
- new net E: J6.11 (Pin_11)
- new net RS: J6.13 (Pin_13)
- new net RW: J6.12 (Pin_12)
- new net V0: J6.14 (Pin_14)
