File: docs/assets/designs/hexapod_circuit/05_ESP32_Sensors.kicad_sch (KiCad schematic)
At the start: 29 parts, among them U3 ESP32, U4 SN65HVD230

Commit message: Add files via upload
Parts:
- added C12, C13: TBD F, symbol Device:C
- R15, R16, R17, R18, R19, R20: value R_US -> TBD Ω
Connections:
- net +3V3_A: now also C12.1
- net +5V_MAIN: now also C13.1
- net GND renamed GND_ELEC
- net GND_ELEC: now also C12.2, C13.2
Other:
- moved on the sheet: C10, C11, C5, C6, C7, C8, C9, R1, R10, R11, R12, R13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

Commit message: upload latest schematic version
Parts:
- removed C12: TBD F, symbol Device:C
- removed R13: TBD Ω, symbol Device:R_US
- removed U4: SN65HVD230, Package_SO:SOIC-8_3.9x4.9mm_P1.27mm, symbol Interface_CAN_LIN:SN65HVD230
- added C12: 100 µF, symbol Device:C_US
- added C14: 0.1 µF, symbol Device:C
- added U4: SN65HVD230, Package_SO:SOIC-8_3.9x4.9mm_P1.27mm, symbol Interface_CAN_LIN:SN65HVD232
- added U5: MPU9250, symbol Connector_Generic:Conn_01x10
- C10, C5, C6, C7, C8, C9: value TBD F -> 10 nF
- C13: value TBD F -> 1 µF
- R1, R2, R3, R4, R5, R6: value FSR -> FSR 402
- R10, R11, R12, R7, R8, R9: value TBD Ω -> 39 kΩ
- R15, R16, R17, R18, R19, R20: value TBD Ω -> 100 Ω
Connections:
- net +3V3_A: now also C14.1, U4.3 (VCC), U5.10 (Pin_10); no longer U3.15 (Pin_15)
- net +5V_MAIN: now also C12.1
- net CAN_H: now also U4.7 (CANH)
- net CAN_L: now also U4.6 (CANL)
- net CAN_RX: now also U4.1 (D)
- net CAN_TX: now also U4.4 (R)
- net D21: now also U5.7 (Pin_7)
- net D23: now also U5.3 (Pin_3)
- net GND_ELEC: now also C12.2, C14.2, U4.2 (GND), U5.4 (Pin_4), U5.9 (Pin_9); no longer U3.14 (Pin_14)
- new net ECL: U5.5 (Pin_5)
- new net EDA: U5.6 (Pin_6)
- new net FSYNC: U5.1 (Pin_1)
- new net NCS: U5.2 (Pin_2)
- new net SCL: U5.8 (Pin_8)
Other:
- note added: "CHECK IF PULL UPS NEEDED"
- moved on the sheet: C10, C11, C13, C5, C6, C7, C8, C9, R1, R10, R11, R12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
